File: Hardware/Bottom/pearwatch-bottom.brd (EAGLE design)
At the start: 38 x 38 mm, 51 parts, among them SW1 SWITCH.MOM, SW2 SWITCH.MOM, U2 NRF52832_MODULE_MDBT42, U4 PCF8523

Commit message: adding bottom board
Parts:
- removed C12: 10u, LinnesLab-Passives:C0805
- removed C13: 2.2uF, LinnesLab-Passives:C0402
- removed C2, C5, C6, C7: 1u, LinnesLab-Passives:C0603
- removed C8, C9: (no value), LinnesLab-Passives:C0603
- removed CHRG2: MCP73831, LinnesLab-Power:SOT23-5
- removed CORTEX1: CORTEX_DEBUG_PTH, LinnesLab-Connectors:2X5-PTH-1.27MM
- removed D1, D4, D5: (no value), LinnesLab-DiscreteSemi:USC
- removed J2: (no value), LinnesLab-Connectors:1X02
- removed L2: 10u, LinnesLab-Passives:L0603
- removed LDO2: MIC5504, LinnesLab-Power:SOT23-5
- removed LED3: RED, LinnesLab-LED:LED-0603
- removed LED4: BLUE, LinnesLab-LED:LED-0603
- removed R11: (no value), LinnesLab-Passives:R0603
- removed R12: 100k, LinnesLab-Passives:R0603
- removed R3, R4: 1k, LinnesLab-Passives:R0603
- removed R5, R6, R8, R9: 10k, LinnesLab-Passives:R0603
- removed R7: 390k, LinnesLab-Passives:R0603
- removed SD2: (no value), LinnesLab-Connectors:MICROSD
- removed SW1, SW2: SWITCH.MOM, LinnesLab-Switches:TACTILE_SWITCH_SMD_6.2MM_TALL
- removed SW3, SW4: (no value), LinnesLab-Switches:BUTTON-GULLWING
- removed U2: NRF52832_MODULE_MDBT42, LinnesLab-Microcontrollers:BLE_MODULE_RAYTAC_MDBT42
- removed U3: (no value), LinnesLab-Displays:UG-2864HSWEG01_0.96IN_NO-WRAPAROUND
- removed U4: PCF8523, LinnesLab-Clocks:SO8
- removed USB2: USB.MICRO-BIGGERPADS, LinnesLab-Connectors:USB-MICRO-01.BIGGERPADS
- removed XTAL2: 32.768kHz, LinnesLab-Clocks:2-SMD.NOLEAD.2.0MMTO1.2MM
- removed XTAL3: 32.7680kHz, LinnesLab-Clocks:2-SMD.NOLEAD.2.0MMTO1.2MM
- added C22, C24: 100n, LinnesLab-Passives:C0603
- added IMU1: LSM6DS3_CAST, LinnesLab-Sensors:LSM6DS3_CAST
- added OP3: (no value), LinnesLab-AnalogIC:SO14
- added OP4: (no value), LinnesLab-AnalogIC:SOT23-5
- added Q1: (no value), LinnesLab-DiscreteSemi:SOT23-3
- added R16: (no value), LinnesLab-Passives:R0603
- added R17, R18: 10k, LinnesLab-Passives:R0402
- added R19, R21: 220k, LinnesLab-Passives:R0603
- added R20, R23: 1M, LinnesLab-Passives:R0603
- added R22: 10M, LinnesLab-Passives:R0603
- added R24: 10k, LinnesLab-Passives:R0603
- added U$3: (no value), LinnesLab-Connectors:PPG.MODULE.2
- added U$4: AD5171, LinnesLab-DigitalIC:SOT-23-8
- added U1: AD5242-SO16, LinnesLab-DigitalIC:SO16
- C10, C11: value 300p -> 100n
- C14: value 100n -> 2.2n
- C15: value 2.2uF -> 2.2u; device LinnesLab-Passives:C0402 -> LinnesLab-Passives:C0603
- C16: value 10uF -> 2.2u
- C17, C18: value 2.2uF -> 100n; device LinnesLab-Passives:C0402 -> LinnesLab-Passives:C0603
- C19: value 2.2uF -> 2.2n; device LinnesLab-Passives:C0402 -> LinnesLab-Passives:C0603
- C20: value 4.7u -> 22u
- C21: value 4.7u -> 22n
- R13, R15: value 100k -> 220k
- R14: value 100k -> 10M
- moved C14 25.3 mm to (25.4, 26.7), turned to 90 degrees
- moved R14 24.7 mm to (26.3, 23.4)
- moved C11 22.1 mm to (13.3, 25.3)
- moved C20 21.6 mm to (31.8, 19.7), turned to 0 degrees
- moved R15 21.0 mm to (19.8, 30.3), turned to 0 degrees
- moved R13 20.4 mm to (23.5, 26.7)
- moved C18 19.3 mm to (7.82, 18.7), turned to 0 degrees
- moved C19 17.6 mm to (27.4, 15.7), turned to 0 degrees
- moved C10 16.4 mm to (25.4, 30.0), turned to 90 degrees
- moved C15 13.9 mm to (23.5, 30.2)
- moved C21 12.9 mm to (31.5, 15.8), turned to 0 degrees
- moved C16 10.8 mm to (20.2, 32.9), turned to 0 degrees
- moved C17 6.24 mm to (8.15, 21.2), turned to 0 degrees
Connections:
- removed net BATT: R13.1, R14.2
- removed net CD1: SD2.CD1
- removed net CD2: SD2.CD2
- removed net CHRG.STAT: CHRG2.1, R12.1
- removed net CS.OLED: U3.13
- removed net DC.OLED: U3.15
- removed net DFU: SW3.3, U2.34
- removed net DTR: C14.1
- removed net FRST: U2.38
- removed net LED1: R3.2, U2.31
- removed net LED2: R4.2, U2.33
- removed net MISO: SD2.7, U2.28
- removed net MOSI: SD2.3, U2.27, U3.19
- removed net N$1: R6.2, U3.11
- removed net N$11: L2.1, U2.10
- removed net N$12: C7.1, L2.2, U2.9
- removed net N$14: CORTEX1.8
- removed net N$2: R7.1, U3.26
- removed net N$3: C13.2, U3.2
- removed net N$4: C8.2, U2.13, XTAL2.P$1
- removed net N$5: C13.1, C14.2, D1.+, R5.1, U3.3
- removed net N$6: C9.1, U2.14, XTAL2.P$2
- removed net N$7: C15.2, U3.4
- removed net P0.09/NFC1: C11.1, U2.22
- removed net P0.10/NFC2: C10.1, U2.23
- removed net RESET: CORTEX1.10, SW4.1, U2.35
- removed net RESET.OLED: U3.14
- removed net RXD: U2.21
- removed net SCK: SD2.5, U2.26, U3.18
- removed net SD.CS: SD2.2
- removed net SWCLK: CORTEX1.4, U2.36
- removed net SWDIO: CORTEX1.2, U2.37
- removed net SWO: CORTEX1.6, U2.32
- removed net TXD: U2.19
- removed net USB+: USB2.3
- removed net USB-: USB2.2
- removed net VBATT: U4.3
- removed net VIN: C21.2, C5.2, CHRG2.4, D4.-, D5.-, LDO2.1, LDO2.3, R12.2
- removed net VLIPO: C20.1, CHRG2.3, D4.+, J2.2, R13.2
- removed net V_USB: D5.+, USB2.1
- new net G.A1: U1.2
- new net G.A2: U1.16
- new net G.O1: U1.1
- new net G.O2: U1.13
- new net G.W2: C21.1, OP3.2, R24.1, U1.15
- new net LED: Q1.3
- new net LED.C: U$3.LD1
- new net LED.CTRL: U$4.8
- new net N$16: C14.1, C16.1, OP3.7, R14.2
- new net N$18: C19.2, OP3.9, R22.1, R23.2
- new net PD.C: C10.1, OP4.4, U$3.PD, U1.4
- new net PPG: C21.2, OP3.1, U1.14
- new net TIA: C10.2, C15.1, OP4.1, U1.3
- new net VREF: OP3.13, OP3.14, OP3.3, R20.1, R23.1
- net 3.3V: now also C11.2, C18.2, C22.2, C24.2, IMU1.2, OP3.4, OP4.5, R13.2, R17.2, U$3.V+, U$4.2, U$4.6, U1.5, U1.6; no longer C12.2, C19.2, C2.1, C6.1, CORTEX1.1, D1.-, LDO2.5, R5.2, R8.2, R9.2, SD2.4, U2.11, U3.6, U3.9, U4.8
- net GND: now also C11.1, C22.1, C24.1, IMU1.1, OP3.11, OP4.2, OP4.3, Q1.2, R18.1, R19.1, R21.1, U$3.GND, U$4.3, U1.10, U1.11, U1.12, U1.9; no longer C10.2, C11.2, C12.1, C16.1, C19.1, C2.2, C20.2, C21.1, C5.1, C6.2, C7.2, C8.1, C9.2, CHRG2.2, CORTEX1.3, CORTEX1.5, CORTEX1.7, CORTEX1.9, J2.1, LDO2.2, LED3.C, LED4.C, R11.1, R14.1, R15.1, R6.1, R7.2, SD2.6, SD2.MT1, SD2.MT2, SW3.1, SW4.3, U2.1, U2.12, U2.24, U2.39, U3.1, U3.10, U3.12, U3.29, U3.30, U3.8, U4.4, USB2.5, USB2.S1, USB2.S2, USB2.S3, USB2.S4, USB2.S5, USB2.S6
- net N$10: now also OP3.12, R17.1, R18.2; no longer LED4.A, R4.1
- net N$13: now also C15.2, OP3.5, R13.1, R19.2; no longer C16.2, U3.28
- net N$15: now also C14.2, OP3.6, R14.1, R20.2; no longer C18.2, U3.27
- net N$17: now also C16.2, OP3.10, R15.1, R21.2; no longer CHRG2.5, R11.2
- net N$19: now also C19.1, C20.1, OP3.8, R22.2; no longer U4.2, XTAL3.P$1
- net N$20: now also C20.2, R24.2; no longer U4.1, XTAL3.P$2
- net N$8: now also Q1.1, R16.2; no longer C15.1, U3.5
- net N$9: now also R16.1, U$4.1, U$4.7; no longer LED3.A, R3.1
- net SCL: now also IMU1.3, U$4.4, U1.7; no longer R8.1, U2.3, U4.6
- net SDA: now also IMU1.4, U$4.5, U1.8; no longer R9.1, U2.2, U4.5
Routing:
- added copper zone on layer 1, net 3.3V
Other:
- board size 38 x 38 mm -> 33 x 33 mm

Commit message: making connections top and bottom board
Parts:
- added J1: (no value), LinnesLab-Connectors:1X07
- moved C16 4.90 mm to (19.8, 28.0)
- moved IMU1 1.80 mm to (14.7, 28.1)
- moved C11 1.31 mm to (13.1, 24.0)
- moved C24 1.21 mm to (8.26, 28.9)
Connections:
- net LED.CTRL renamed D29/LED.CTRL
- removed net TIA: C10.2, C15.1, OP4.1, U1.3
- new net A6/TIA: C10.2, C15.1, J1.5, OP4.1, U1.3
- new net A7/PPG: C21.2, J1.7, OP3.1
- new net D29/LED.CTR: J1.6
- net PPG: no longer C21.2, OP3.1
Changed lines of the file:
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@@
 <setting verticaltext="up"/>
 </settings>
-<grid distance="1" unitdist="mil" unit="mil" style="lines" multiple="1" display="no" altdistance="5" altunitdist="mil" altunit="mil"/>
+<grid distance="1" unitdist="mil" unit="mm" style="lines" multiple="1" display="no" altdistance="5" altunitdist="mil" altunit="mil"/>
 <layers>
 <layer number="1" name="Top" color="4" fill="1" visible="yes" active="yes"/>
@@
 <attribute name="VALUE" x="27.3304" y="29.3624" size="1.27" layer="27" rot="R90"/>
 </element>
-<element name="C11" library="LinnesLab-Passives" package="C0603" value="100n" x="13.335" y="25.273" smashed="yes">
-<attribute name="NAME" x="12.7" y="25.908" size="0.6604" layer="25"/>
-<attribute name="VALUE" x="12.7" y="23.368" size="1.27" layer="27"/>
+<element name="C11" library="LinnesLab-Passives" package="C0603" value="100n" x="13.1318" y="23.9776" smashed="yes">
+<attribute name="NAME" x="12.4968" y="24.6126" size="0.6604" layer="25"/>
+<attribute name="VALUE" x="12.4968" y="22.0726" size="1.27" layer="27"/>
 </element>
 <element name="U$4" library="LinnesLab-DigitalIC" package="SOT-23-8" package3d_urn="urn:adsk.eagle:package:17879439/2" value="AD5171" x="7.7978" y="13.843" smashed="yes">
@@
 <attribute name="VALUE" x="25.4254" y="29.5402" size="1.27" layer="27" rot="R90"/>
 </element>
-<element name="C16" library="LinnesLab-Passives" package="C0603" value="2.2u" x="20.2438" y="32.8676" smashed="yes">
-<attribute name="NAME" x="19.6088" y="33.5026" size="0.6604" layer="25"/>
-<attribute name="VALUE" x="19.6088" y="30.9626" size="1.27" layer="27"/>
+<element name="C16" library="LinnesLab-Passives" package="C0603" value="2.2u" x="19.7612" y="27.9908" smashed="yes">
+<attribute name="NAME" x="19.1262" y="28.6258" size="0.6604" layer="25"/>
+<attribute name="VALUE" x="19.1262" y="26.0858" size="1.27" layer="27"/>
 </element>
 <element name="R15" library="LinnesLab-Passives" package="R0603" package3d_urn="urn:adsk.eagle:package:15661944/2" value="220k" x="19.8374" y="30.3276" smashed="yes">
@@
 <attribute name="VALUE" x="30.3022" y="11.9888" size="1.27" layer="27"/>
 </element>
-<element name="IMU1" library="LinnesLab-Sensors" package="LSM6DS3_CAST" value="LSM6DS3_CAST" x="14.9352" y="29.8704" smashed="yes">
-<attribute name="NAME" x="12.3952" y="33.0454" size="0.6604" layer="25"/>
-<attribute name="VALUE" x="12.3952" y="25.4254" size="0.6604" layer="27"/>
-</element>
-<element name="C24" library="LinnesLab-Passives" package="C0603" value="100n" x="8.5852" y="30.0228" smashed="yes" rot="R270">
-<attribute name="NAME" x="9.2202" y="30.6578" size="0.6604" layer="25" rot="R270"/>
-<attribute name="VALUE" x="6.6802" y="30.6578" size="0.6604" layer="27" rot="R270"/>
+<element name="IMU1" library="LinnesLab-Sensors" package="LSM6DS3_CAST" value="LSM6DS3_CAST" x="14.6812" y="28.0924" smashed="yes">
+<attribute name="NAME" x="12.1412" y="31.2674" size="0.6604" layer="25"/>
+<attribute name="VALUE" x="12.1412" y="23.6474" size="0.6604" layer="27"/>
+</element>
+<element name="C24" library="LinnesLab-Passives" package="C0603" value="100n" x="8.255" y="28.8544" smashed="yes" rot="R270">
+<attribute name="NAME" x="8.89" y="29.4894" size="0.6604" layer="25" rot="R270"/>
+<attribute name="VALUE" x="6.35" y="29.4894" size="0.6604" layer="27" rot="R270"/>
+</element>
+<element name="J1" library="LinnesLab-Connectors" package="1X07" value="" x="5" y="33" smashed="yes">
+<attribute name="NAME" x="4.6444" y="33.508" size="0.6096" layer="25" font="vector" ratio="20"/>
+<attribute name="VALUE" x="3.73" y="30.968" size="0.6096" layer="27" font="vector" ratio="20"/>
 </element>
 </elements>
@@
 <wire x1="33.8328" y1="10.9982" x2="32.5628" y2="10.9982" width="0" layer="19" extent="1-1"/>
 <wire x1="20.27" y1="24.08" x2="26.4296" y2="19.8628" width="0" layer="19" extent="1-1"/>
-<wire x1="12.485" y1="25.273" x2="20.27" y2="24.08" width="0" layer="19" extent="1-1"/>
-<wire x1="7.3256" y1="23.7998" x2="12.485" y2="25.273" width="0" layer="19" extent="1-1"/>
+<wire x1="12.2818" y1="23.9776" x2="20.27" y2="24.08" width="0" layer="19" extent="1-1"/>
+<wire x1="7.3256" y1="23.7998" x2="12.2818" y2="23.9776" width="0" layer="19" extent="1-1"/>
 <wire x1="7.3034" y1="21.209" x2="7.3256" y2="23.7998" width="0" layer="19" extent="1-1"/>
 <wire x1="6.9732" y1="18.7198" x2="7.3034" y2="21.209" width="0" layer="19" extent="1-1"/>
-<wire x1="12.3952" y1="31.1404" x2="12.485" y2="25.273" width="0" layer="19" extent="1-1"/>
-<wire x1="8.5852" y1="30.8728" x2="12.3952" y2="31.1404" width="0" layer="19" extent="1-1"/>
+<wire x1="12.1412" y1="29.3624" x2="12.2818" y2="23.9776" width="0" layer="19" extent="1-1"/>
+<wire x1="8.255" y1="29.7044" x2="12.1412" y2="29.3624" width="0" layer="19" extent="1-1"/>
 <wire x1="8.1072" y1="12.6666" x2="6.9732" y2="18.7198" width="0" layer="19" extent="1-1"/>
 <wire x1="8.57" y1="9.4394" x2="8.1072" y2="12.6666" width="0" layer="19" extent="1-1"/>
@@
 <contactref element="U1" pad="8"/>
 <contactref element="IMU1" pad="4"/>
-<wire x1="8.7572" y1="15.0194" x2="17.4752" y2="31.1404" width="0" layer="19" extent="1-1"/>
+<wire x1="8.7572" y1="15.0194" x2="17.2212" y2="29.3624" width="0" layer="19" extent="1-1"/>
 <wire x1="33.8328" y1="4.8514" x2="8.7572" y2="15.0194" width="0" layer="19" extent="1-1"/>
 </signal>
@@
 <contactref element="U1" pad="7"/>
 <contactref element="IMU1" pad="3"/>
-<wire x1="8.7572" y1="12.6666" x2="17.4752" y2="28.6004" width="0" layer="19" extent="1-1"/>
+<wire x1="8.7572" y1="12.6666" x2="17.2212" y2="26.8224" width="0" layer="19" extent="1-1"/>
 <wire x1="32.5628" y1="4.8514" x2="8.7572" y2="12.6666" width="0" layer="19" extent="1-1"/>
 </signal>
-<signal name="TIA">
+<signal name="A6/TIA">
 <contactref element="C10" pad="2"/>
 <contactref element="U1" pad="3"/>
 <contactref element="C15" pad="1"/>
 <contactref element="OP4" pad="1"/>
+<contactref element="J1" pad="5"/>
 <wire x1="23.5204" y1="29.3252" x2="25.4254" y2="30.8474" width="0" layer="19" extent="1-1"/>
+<wire x1="15.16" y1="33" x2="23.5204" y2="29.3252" width="0" layer="19" extent="1-1"/>
 <wire x1="31.1048" y1="21.681" x2="23.5204" y2="29.3252" width="0" layer="19" extent="1-1"/>
 <wire x1="27.4828" y1="4.8514" x2="31.1048" y2="21.681" width="0" layer="19" extent="1-1"/>
@@
 <wire x1="6.8072" y1="12.6666" x2="7.4572" y2="15.0194" width="0" layer="19" extent="1-1"/>
 </signal>
-<signal name="LED.CTRL">
+<signal name="D29/LED.CTRL">
 <contactref element="U$4" pad="8"/>
 </signal>
@@
 <signal name="PPG">
 <contactref element="U1" pad="14"/>
-<contactref element="C21" pad="2"/>
-<contactref element="OP3" pad="1"/>
-<wire x1="32.3968" y1="15.7988" x2="28.1848" y2="33.782" width="0" layer="19" extent="1-1"/>
-<wire x1="27.4828" y1="10.9982" x2="32.3968" y2="15.7988" width="0" layer="19" extent="1-1"/>
 </signal>
 <signal name="N$13">
@@
 <wire x1="26.3144" y1="24.218" x2="28.1848" y2="26.162" width="0" layer="19" extent="1-1"/>
 <wire x1="25.3746" y1="25.82" x2="26.3144" y2="24.218" width="0" layer="19" extent="1-1"/>
-<wire x1="19.3938" y1="32.8676" x2="25.3746" y2="25.82" width="0" layer="19" extent="1-1"/>
+<wire x1="18.9112" y1="27.9908" x2="25.3746" y2="25.82" width="0" layer="19" extent="1-1"/>
 </signal>
 <signal name="N$17">
@@
 <contactref element="OP3" pad="10"/>
 <wire x1="28.1296" y1="19.8628" x2="33.3848" y2="28.702" width="0" layer="19" extent="1-1"/>
-<wire x1="21.0938" y1="32.8676" x2="33.3848" y2="28.702" width="0" layer="19" extent="1-1"/>
-<wire x1="18.9874" y1="30.3276" x2="21.0938" y2="32.8676" width="0" layer="19" extent="1-1"/>
+<wire x1="20.6112" y1="27.9908" x2="33.3848" y2="28.702" width="0" layer="19" extent="1-1"/>
+<wire x1="18.9874" y1="30.3276" x2="20.6112" y2="27.9908" width="0" layer="19" extent="1-1"/>
 </signal>
 <signal name="N$18">
@@
 <wire x1="32.5238" y1="17.7546" x2="32.6" y2="19.6596" width="0" layer="19" extent="1-1"/>
 </signal>
+<signal name="A7/PPG">
+<contactref element="C21" pad="2"/>
+<contactref element="OP3" pad="1"/>
+<contactref element="J1" pad="7"/>
+<wire x1="20.24" y1="33" x2="28.1848" y2="33.782" width="0" layer="19" extent="1-1"/>
+<wire x1="32.3968" y1="15.7988" x2="28.1848" y2="33.782" width="0" layer="19" extent="1-1"/>
+</signal>
+<signal name="D29/LED.CTR">
+<contactref element="J1" pad="6"/>
+</signal>
 </signals>
