File: Hardware/Top/pearwatch-TOP.sch (EAGLE design)
At the start: 51 parts, among them SW1 SWITCH.MOM, SW2 SWITCH.MOM, U2 FT231XS, U3 PCF8523, U5 NRF52832_MODULE_MDBT42

Commit message: making connections top and bottom board
Parts:
- added J1: (no value), LinnesLab-Connectors:CONN_07
- renumbered SW1 to D11/SW1, SW2 to D15/SW2
Connections:
- removed net DC.OLED: U6.DC/I2C_SA0
- removed net RESET.OLED: U6./RES
- removed net SD.CS: SD2.CS
- new net A4/BATT: U5.P0.28/AIN4
- new net A6/TIA: U5.P0.30/AIN6
- new net A7/PPG: U5.P0.31/AIN7
- new net D11/SW1: U5.P0.11
- new net D15/SW2: U5.P0.15
- new net D27/CHRG.STATUS: U5.P0.27
- new net D29/LED.CTRL: U5.P0.29/AIN5
- new net D3/RESET.OLED: U5.P0.03/AIN1, U6./RES
- new net D4/DC.OLED: U5.P0.04/AIN2, U6.DC/I2C_SA0
- new net D7/SD.CS: SD2.CS, U5.P0.07
Changed lines of the file:
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@@
 <part name="GND22" library="LinnesLab-Symbols" deviceset="GND" device=""/>
 <part name="SD2" library="LinnesLab-Connectors" deviceset="MICROSD" device="" package3d_urn="urn:adsk.eagle:package:17873109/2"/>
-<part name="SW1" library="LinnesLab-Switches" deviceset="SWITCH.MOM" device=""/>
-<part name="SW2" library="LinnesLab-Switches" deviceset="SWITCH.MOM" device=""/>
+<part name="D11/SW1" library="LinnesLab-Switches" deviceset="SWITCH.MOM" device=""/>
+<part name="D15/SW2" library="LinnesLab-Switches" deviceset="SWITCH.MOM" device=""/>
 <part name="GND51" library="LinnesLab-Symbols" deviceset="GND" device=""/>
 <part name="GND52" library="LinnesLab-Symbols" deviceset="GND" device=""/>
@@
 <part name="SUPPLY1" library="LinnesLab-Symbols" deviceset="3.3V" device=""/>
 <part name="SUPPLY2" library="LinnesLab-Symbols" deviceset="3.3V" device=""/>
+<part name="J1" library="LinnesLab-Connectors" deviceset="CONN_07" device=""/>
 </parts>
 <sheets>
@@
 <attribute name="VALUE" x="119.38" y="-36.83" size="1.778" layer="96"/>
 </instance>
-<instance part="SW1" gate="G$1" x="162.56" y="-10.16" smashed="yes">
+<instance part="D11/SW1" gate="G$1" x="162.56" y="-10.16" smashed="yes">
 <attribute name="NAME" x="162.56" y="-5.334" size="1.778" layer="95" font="vector" align="bottom-center"/>
 <attribute name="VALUE" x="73.66" y="25.146" size="1.778" layer="96" font="vector" align="top-center"/>
 </instance>
-<instance part="SW2" gate="G$1" x="182.88" y="-10.16" smashed="yes">
+<instance part="D15/SW2" gate="G$1" x="182.88" y="-10.16" smashed="yes">
 <attribute name="NAME" x="182.88" y="-5.334" size="1.778" layer="95" font="vector" align="bottom-center"/>
 <attribute name="VALUE" x="182.88" y="-12.954" size="1.778" layer="96" font="vector" align="top-center"/>
@@
 <instance part="SUPPLY2" gate="G$1" x="-40.64" y="116.84" smashed="yes">
 <attribute name="VALUE" x="-40.64" y="119.634" size="1.778" layer="96" align="bottom-center"/>
+</instance>
+<instance part="J1" gate="G$1" x="-144.78" y="-68.58" smashed="yes">
+<attribute name="VALUE" x="-149.86" y="-78.486" size="1.778" layer="96" font="vector"/>
+<attribute name="NAME" x="-149.86" y="-55.372" size="1.778" layer="95" font="vector"/>
 </instance>
 </instances>
@@
 </segment>
 </net>
-<net name="DC.OLED" class="0">
-<segment>
-<label x="144.78" y="71.12" size="1.778" layer="95"/>
-<pinref part="U6" gate="G$1" pin="DC/I2C_SA0"/>
-<wire x1="170.18" y1="71.12" x2="144.78" y2="71.12" width="0.1524" layer="91"/>
-</segment>
-</net>
-<net name="RESET.OLED" class="0">
-<segment>
-<label x="144.78" y="73.66" size="1.778" layer="95"/>
-<pinref part="U6" gate="G$1" pin="/RES"/>
-<wire x1="170.18" y1="73.66" x2="144.78" y2="73.66" width="0.1524" layer="91"/>
-</segment>
-</net>
 <net name="CS.OLED" class="0">
 <segment>
@@
 <label x="93.98" y="-40.64" size="1.27" layer="95" rot="R180" xref="yes"/>
 <pinref part="SD2" gate="G$1" pin="CARD_DETECT"/>
-</segment>
-</net>
-<net name="SD.CS" class="0">
-<segment>
-<wire x1="93.98" y1="-58.42" x2="99.06" y2="-58.42" width="0.1524" layer="91"/>
-<label x="93.98" y="-58.42" size="1.27" layer="95" rot="R180" xref="yes"/>
-<pinref part="SD2" gate="G$1" pin="CS"/>
 </segment>
 </net>
@@
 </segment>
 </net>
+<net name="D7/SD.CS" class="0">
+<segment>
+<pinref part="U5" gate="G$1" pin="P0.07"/>
+<wire x1="5.08" y1="43.18" x2="5.08" y2="40.64" width="0.1524" layer="91"/>
+<label x="5.08" y="40.64" size="1.778" layer="95" rot="R270"/>
+</segment>
+<segment>
+<wire x1="93.98" y1="-58.42" x2="99.06" y2="-58.42" width="0.1524" layer="91"/>
+<label x="93.98" y="-58.42" size="1.27" layer="95" rot="R180" xref="yes"/>
+<pinref part="SD2" gate="G$1" pin="CS"/>
+</segment>
+</net>
+<net name="D11/SW1" class="0">
+<segment>
+<pinref part="U5" gate="G$1" pin="P0.11"/>
+<wire x1="22.86" y1="55.88" x2="25.4" y2="55.88" width="0.1524" layer="91"/>
+<label x="25.4" y="55.88" size="1.778" layer="95"/>
+</segment>
+</net>
+<net name="D15/SW2" class="0">
+<segment>
+<pinref part="U5" gate="G$1" pin="P0.15"/>
+<wire x1="22.86" y1="66.04" x2="25.4" y2="66.04" width="0.1524" layer="91"/>
+<label x="25.4" y="66.04" size="1.778" layer="95"/>
+</segment>
+</net>
+<net name="D3/RESET.OLED" class="0">
+<segment>
+<pinref part="U5" gate="G$1" pin="P0.03/AIN1"/>
+<wire x1="-5.08" y1="43.18" x2="-5.08" y2="40.64" width="0.1524" layer="91"/>
+<label x="-5.08" y="40.64" size="1.778" layer="95"/>
+</segment>
+<segment>
+<label x="144.78" y="73.66" size="1.778" layer="95"/>
+<pinref part="U6" gate="G$1" pin="/RES"/>
+<wire x1="170.18" y1="73.66" x2="144.78" y2="73.66" width="0.1524" layer="91"/>
+</segment>
+</net>
+<net name="D4/DC.OLED" class="0">
+<segment>
+<pinref part="U5" gate="G$1" pin="P0.04/AIN2"/>
+<wire x1="-2.54" y1="43.18" x2="-2.54" y2="38.1" width="0.1524" layer="91"/>
+<label x="-2.54" y="38.1" size="1.778" layer="95"/>
+</segment>
+<segment>
+<label x="144.78" y="71.12" size="1.778" layer="95"/>
+<pinref part="U6" gate="G$1" pin="DC/I2C_SA0"/>
+<wire x1="170.18" y1="71.12" x2="144.78" y2="71.12" width="0.1524" layer="91"/>
+</segment>
+</net>
+<net name="D27/CHRG.STATUS" class="0">
+<segment>
+<pinref part="U5" gate="G$1" pin="P0.27"/>
+<wire x1="-22.86" y1="76.2" x2="-25.4" y2="76.2" width="0.1524" layer="91"/>
+<label x="-30.48" y="76.2" size="1.778" layer="95"/>
+</segment>
+</net>
+<net name="A4/BATT" class="0">
+<segment>
+<pinref part="U5" gate="G$1" pin="P0.28/AIN4"/>
+<wire x1="-22.86" y1="73.66" x2="-25.4" y2="73.66" width="0.1524" layer="91"/>
+<label x="-25.4" y="73.66" size="1.778" layer="95"/>
+</segment>
+</net>
+<net name="D29/LED.CTRL" class="0">
+<segment>
+<pinref part="U5" gate="G$1" pin="P0.29/AIN5"/>
+<wire x1="-22.86" y1="71.12" x2="-25.4" y2="71.12" width="0.1524" layer="91"/>
+<label x="-25.4" y="71.12" size="1.778" layer="95"/>
+</segment>
+</net>
+<net name="A6/TIA" class="0">
+<segment>
+<pinref part="U5" gate="G$1" pin="P0.30/AIN6"/>
+<wire x1="-22.86" y1="68.58" x2="-25.4" y2="68.58" width="0.1524" layer="91"/>
+<label x="-25.4" y="68.58" size="1.778" layer="95"/>
+</segment>
+</net>
+<net name="A7/PPG" class="0">
+<segment>
+<pinref part="U5" gate="G$1" pin="P0.31/AIN7"/>
+<wire x1="-22.86" y1="66.04" x2="-25.4" y2="66.04" width="0.1524" layer="91"/>
+<label x="-25.4" y="66.04" size="1.778" layer="95"/>
+</segment>
+</net>
